File: TEST_Kicad/TEST.kicad_sch (KiCad schematic)
At the start: 25 parts, among them J1_guitare_entrée1 NRJ6HF, J2_guitare_sortie1 NRJ6HF, U1 LM7805_TO220, U3 LM324M_NOPB, U4 SGTL5000XNAA3, U5 IS42S16400J-xC

Commit message: Add files via upload
Parts:
- removed R4: 10k, symbol Device:R
- added C12, C13, C14, C15, C16, C17, C18, C321 (x3): 100nF, Capacitor_SMD:C_0603_1608Metric, symbol Device:C_Small
- added C3, C37, C38, C39, C4, C9: C, symbol Device:C
- added C301, C302: 10pF, Capacitor_SMD:C_0603_1608Metric, symbol Device:C_Small
- added C5, C6: 10uF, Capacitor_SMD:C_0603_1608Metric_Pad1.08x0.95mm_HandSolder, symbol Device:C
- added C7, C8: 22uF, Capacitor_SMD:C_0603_1608Metric_Pad1.08x0.95mm_HandSolder, symbol Device:C
- added J1: Barrel_Jack, symbol Connector:Barrel_Jack
- added L1: 1u, symbol Device:L
- added R302: 10R, Resistor_SMD:R_0603_1608Metric, symbol Device:R_Small
- added R6: 1meg, symbol Device:R
- added R7: 10k, symbol Device:R
- added R8: 470k, symbol Device:R
- added RV11: R_Potentiometer, symbol Device:R_Potentiometer
- added U2: L78L05_SO8, Package_SO:SOIC-8_3.9x4.9mm_P1.27mm, symbol Regulator_Linear:L78L05_SO8
- added U7: MCP6002-I/P, PDIP8_300MC_MCH, symbol 2023-11-07_21-38-13:MCP6002-I_P
- added Y301: 16MHz, Crystal:Crystal_SMD_EuroQuartz_MT-4Pin_3.2x2.5mm, symbol Device:Crystal_GND24_Small
- R5: value 19412 -> 1.2meg
Connections:
- net +1V0: now also C5.1, L1.1; no longer C10.1, U1.1 (VI)
- net GND: now also J2_guitare_sortie1.R, J2_guitare_sortie1.RN, J2_guitare_sortie1.SN, R5.1, C12.2, C13.2, C14.2, C15.2, C16.2, C17.2, C18.2, C301.1, C302.1, C321.2, C321.2, C321.2, C38.2, C39.2, C4.2, C9.2, R6.1, U7.4 (VSS), Y301.2, Y301.4
- net GNDPWR: now also C5.2, C6.2, C7.2, C8.2, U2.2 (GND), U2.3 (GND), U2.6 (GND), U2.7 (GND); no longer R5.2
- net Ve_guitare: now also U7.3 (VINA+)
- net Vs_3,3V: now also U4.20 (VDDIO), C12.1, C13.1, C14.1, C15.1, C16.1, C17.1, C18.1, C321.1, C321.1, C321.1; no longer R5.1
- net Vs_5V: now also C9.1, RV11.1; no longer C11.1, U1.3 (VO)
- net Vs_préampli: now also C37.2, C39.1, R8.1
- net Vs_audio: now reaches U4.11 (LINEOUT_R)
- net Vs_audio: now also U3.13 (IN4+)
- net SYS_MCLK: now reaches U4.21 (SYS_MCLK)
- net DOUT_I2S: now reaches U4.25 (I2S_DOUT)
- net Vs_ampli: now reaches J2_guitare_sortie1.T
- net Vs_ampli: now also J2_guitare_sortie1.TN, U3.14 (OUT4), C4.1, R7.2
- net at U3.12 (IN4-): now also C3.2, R6.2, RV11.3
- new net: C37.1, R5.2, R8.2, U7.1 (VOUTA), U7.2 (VINA-)
- new net: C3.1, R7.1, RV11.2
- new net: C6.1, L1.2, U2.8 (IN)
- new net OSC_IN: C301.2, Y301.3
- new net OSC_OUT: R302.2
- new net V_3,3V: C11.1, U1.3 (VO)
- new net V_5V: C10.1, C38.1, C7.1, C8.1, U1.1 (VI), U2.1 (OUT), U7.8 (VDD)
- new net XTAL_OUT: C302.2, R302.1, Y301.1
- no-connect marks 14 -> 17
Other:
- removed sheet USB_OTG
- note added: "Power Section"
- note added: "Préamplifier & Amplifier"
- note added: "SYSMCLK est connecté a la clock du µP"
- note removed: "Power Board"
- note removed: "Pré-ampli"
- moved on the sheet: C1, C10, C11, C2, J1_guitare_entrée1, J2_guitare_sortie1, R1, R2, R3, RV1, RV10, RV2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

Commit message: Add files via upload
Parts:
- removed C1, C2, C3, C4, C9: C, symbol Device:C
- removed C301, C302: 10pF, Capacitor_SMD:C_0603_1608Metric, symbol Device:C_Small
- removed J1: Barrel_Jack, symbol Connector:Barrel_Jack
- removed J2_guitare_sortie1: NRJ6HF, NRJ6HF:NEUTRIK_NRJ6HF, symbol NRJ6HF:NRJ6HF
- removed L1: 1u, symbol Device:L
- removed R1: 470k, symbol Device:R
- removed R2: 1.2meg, symbol Device:R
- removed R302: 10R, Resistor_SMD:R_0603_1608Metric, symbol Device:R_Small
- removed R6: 1meg, symbol Device:R
- removed R7: 10k, symbol Device:R
- removed RV11: R_Potentiometer, symbol Device:R_Potentiometer
- removed U2: L78L05_SO8, Package_SO:SOIC-8_3.9x4.9mm_P1.27mm, symbol Regulator_Linear:L78L05_SO8
- removed U3: LM324M_NOPB, LM324M_NOPB:SOIC127P600X175-14N, symbol LM324M_NOPB:LM324M_NOPB
- removed Y301: 16MHz, Crystal:Crystal_SMD_EuroQuartz_MT-4Pin_3.2x2.5mm, symbol Device:Crystal_GND24_Small
- added J2: 4840.2201, CONN_4840.2201_SCH, symbol 2023-11-07_22-49-07:4840.2201
- added J2_guitare_sortie: NRJ6HF, NRJ6HF:NEUTRIK_NRJ6HF, symbol NRJ6HF:NRJ6HF
- added J3: 173950578, CONN3_950578_WRE, symbol Regulator 5V:173950578
- added R4: 1meg, symbol Device:R
- added R9: 10k, symbol Device:R
- added RV12: R_Potentiometer, symbol Device:R_Potentiometer
- C5: value 10uF -> C; footprint Capacitor_SMD:C_0603_1608Metric_Pad1.08x0.95mm_HandSolder -> (none)
- C6: value 10uF -> 100uF
- C7: value 22uF -> 100µF
- C8: value 22uF -> C; footprint Capacitor_SMD:C_0603_1608Metric_Pad1.08x0.95mm_HandSolder -> (none)
- renumbered J1_guitare_entrée1 to J1_guitare_entrée
Connections:
- net +1V0: now also C6.1, J2.1, J3.1; no longer C5.1
- net GND: now also C8.2, J2_guitare_sortie.S, R4.1
- net GNDPWR: now also J2.2, J3.2; no longer C5.2, C8.2
- net V_5V: now also J3.3; no longer C8.1
- net Vs_5V: now also RV12.1
- net Vs_ampli: now also C8.1, J2_guitare_sortie.T, R9.2
- net Vs_audio: now also U7.5 (VINB+)
- net at U7.6 (VINB-): now also C5.2, R4.2, RV12.3
- new net: C5.1, R9.1, RV12.2
- new net Earth: J2.3
- no-connect marks 17 -> 15
Other:
- sheet stm32 ports: added DOUT_I2C, PA8; removed none
- note added: "STM32"
- moved on the sheet: C10, C11, C12, C13, C14, C15, C16, C17, C18, C321, C37, C38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
