File: TEST_Kicad/stm32.kicad_sch (KiCad schematic)
At the start: 1 part, among them U6 STM32F446ZCTx

Commit message: Add files via upload
Parts:
- added C304 (x13): 1uF, Capacitor_SMD:C_0603_1608Metric, symbol Device:C_Small
Connections:
- net VDD: now also U6.6 (VBAT), U6.95 (VDDUSB), C304.1, C304.1, C304.1, C304.1, C304.1, C304.1, C304.1, C304.1, C304.1, C304.1, C304.1, C304.1, C304.1
- new net GND: C304.2, C304.2, C304.2, C304.2, C304.2, C304.2, C304.2, C304.2, C304.2, C304.2, C304.2, C304.2, C304.2

Commit message: Add files via upload
Connections:
- net PA8: now reaches U6.100 (PA8)
- net DOUT_I2C: now reaches U6.140 (PB9)
Changed lines of the file:
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@@
+    (effects (font (size 1.27 1.27)) (justify left))
+  )
+  (hierarchical_label "DOUT_I2C" (shape input) (at 229.87 123.19 0) (fields_autoplaced)
     (effects (font (size 1.27 1.27)) (justify left))
   )
@@
     (effects (font (size 1.27 1.27)) (justify left))
   )
+  (hierarchical_label "PA8" (shape input) (at 229.87 77.47 0) (fields_autoplaced)
+    (effects (font (size 1.27 1.27)) (justify left))
+  )
