File: Electronic Board/TEST.kicad_sch (KiCad schematic)
At the start: 39 parts, among them J1_guitare_entrée1 NRJ6HF, J2 4840.2201, J2_guitare_sortie1 NRJ6HF, J3 173950578, U1 LM7805_TO220, U4 SGTL5000XNAA3, U5 IS42S16400J-xC

Commit message: Add files via upload
Parts:
- removed C321 (x2): 100nF, Capacitor_SMD:C_0201_0603Metric_Pad0.64x0.40mm_HandSolder, symbol Device:C_Small
- removed J1_guitare_entrée1, J2_guitare_sortie1: NRJ6HF, NRJ6HF:NEUTRIK_NRJ6HF, symbol NRJ6HF:NRJ6HF
- added C11, C12, C30, C321, C34, C35, C36, C37, C38, C8, C9: 100nF, Capacitor_SMD:C_0201_0603Metric_Pad0.64x0.40mm_HandSolder, symbol Device:C_Small
- added C6, C7: 1uF, Capacitor_SMD:C_0603_1608Metric, symbol Device:C_Small
- added D2: LED, LED_SMD:LED_0201_0603Metric_Pad0.64x0.40mm_HandSolder, symbol Device:LED
- added J1_guitare_entrée1, J2_guitare_sortie1: NRJ6HF, Connector_Audio:Jack_6.35mm_Neutrik_NRJ6HF_Horizontal, symbol Connector_Audio:NRJ6HF
- added R3: 330, Resistor_SMD:R_0201_0603Metric_Pad0.64x0.40mm_HandSolder, symbol Device:R
- added SW2: SW_SPDT, Library:RS_Pro_SPDT_8466720, symbol Switch:SW_SPDT
- added U2: BU18SD2MG-MTR, Package_TO_SOT_SMD:SOT-23-5, symbol WITNS_ROHM:BU18SD2MG-MTR
- J2: footprint CONN_4840.2201_SCH -> Library:Regulator4840-2201
- J3: footprint CONN3_950578_WRE -> Library:CONN3_950578_WRE_173950578
- RV1, RV10, RV2, RV3, RV4, RV5, RV6, RV7, RV8, RV9: value R_Potentiometer -> 100k; footprint (none) -> Library:Potentiometer_Alpha_RD901F-40-00D_Single_Vertical
Connections:
- net +3.3V: now also C321.1, C6.1, SW2.2 (B), U2.1 (IN), U2.3 (STBY); no longer RV2.1, RV3.1, RV6.1, U4.30 (VDDD)
- net GND: now also U4.31 (CTRL_ADR0_CS), U4.32 (CTRL_MODE), C11.2, C12.2, C30.2, C321.2, C34.2, C35.2, C36.2, C37.2, C38.2, C6.2, C7.2, C8.2, C9.2, J1_guitare_entrée1.S, J2_guitare_sortie1.S, SW2.3 (C), U2.2 (GND)
- net Pot_0: now also C30.1
- net Pot_1: now also C8.1
- net Pot_2: now also C9.1
- net Pot_3: now also C11.1
- net Pot_4: now also C12.1
- net Pot_5: now also C34.1
- net Pot_6: now also C35.1
- net Pot_7: now also C36.1
- net Pot_8: now also C37.1
- net Pot_9: now also C38.1
- net Ve_guitare_L: now also J1_guitare_entrée1.T
- net Ve_guitare_R: now also J1_guitare_entrée1.R
- net Vs_guitare_L: now also J2_guitare_sortie1.T
- net Vs_guitare_R: now also J2_guitare_sortie1.R
- new net: R3.2, SW2.1 (A)
- new net: D2.2 (A), R3.1
- new net +1V8: C7.1, U2.5 (OUT)
- new net Buffer: D2.1 (K)
- no-connect marks 26 -> 24
Other:
- sheet stm32 ports: added Buffer; removed none
- note added: "Buffer Button"
- note added: "Linear Regulator"
- note added: "Switch Regulator"
- note removed: "I2S DOUT : transmettre les données audio numériques vers d'autres composants ou périphériques, comme des amplificateurs audio, des convertisseurs numérique-analogique (DAC), des processeurs de traitement audio, etc."
- note removed: "SYSMCLK est connecté a la clock du µP"
- moved on the sheet: C20, C321, H1, H2, H3, H4, R3, RV1, RV2, RV3, RV4, RV5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

Commit message: Add files via upload
Parts:
- removed C3: 10uF, Capacitor_SMD:C_0201_0603Metric_Pad0.64x0.40mm_HandSolder, symbol Device:C
- removed C4: 1uF, Capacitor_SMD:C_0201_0603Metric_Pad0.64x0.40mm_HandSolder, symbol Device:C
- removed D1: LED, LED_SMD:LED_0201_0603Metric_Pad0.64x0.40mm_HandSolder, symbol Device:LED
- removed R3: 1k, Resistor_SMD:R_0201_0603Metric_Pad0.64x0.40mm_HandSolder, symbol Device:R
- removed U1: LM7805_TO220, Package_TO_SOT_THT:TO-220-3_Vertical, symbol Regulator_Linear:LM7805_TO220
- added C502, C505: 1uF, Capacitor_SMD:C_0603_1608Metric, symbol Device:C_Small
- added D502: RED, LED_SMD:LED_0603_1608Metric, symbol Device:LED_Small
- added R502: 1k, Resistor_SMD:R_0603_1608Metric, symbol Device:R_Small
- added TP1, TP10, TP11, TP12, TP2, TP3, TP4, TP5, TP6, TP7, TP8, TP9: TestPoint, TestPoint:TestPoint_Pad_D1.5mm, symbol Connector:TestPoint
- added U502: BU33SD5WG-TR, Package_TO_SOT_SMD:SOT-23-5, symbol WITNS_ROHM:BU33SD5WG-TR
- renumbered C30 to C40
Connections:
- net +1V8: now also TP2.1
- net +3.3V: now also RV2.1, RV3.1, RV6.1, C505.1, D502.2 (A), TP1.1, U502.5 (OUT)
- net +5V: now also C502.1, TP12.1, U502.1 (IN), U502.3 (STBY)
- net CK_I2S: now also TP5.1
- net DOUT_I2S: now also TP6.1
- net GND: now also C502.2, C505.2, R502.2, U502.2 (GND)
- net SCL_I2C: now also TP9.1
- net SDA_I2C: now also TP8.1
- net SD_I2S: now also TP7.1
- net SYS_MCLK: now also TP3.1
- net Ve_guitare_R: now also TP10.1
- net Vs_guitare_R: now also TP11.1
- net WS_I2S: now also TP4.1
- new net LED33_MID: D502.1 (K), R502.1
Other:
- note removed: "Linear Regulator"
- moved on the sheet: C1, C11, C12, C13, C14, C15, C16, C17, C18, C19, C2, C20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
