File: Electronic Board/_autosave-EC.kicad_pcb (KiCad board)
At the start: 6 copper layers, 169 x 100.2 mm, 113 parts, among them J1 NMJ4HCD2, J2 4840.2201, J3 173950578, J4 NMJ4HCD2, J5 NMJ4HCD2, J6 NMJ4HCD2, J7 Conn_01x03, J8 Conn_02x07_Odd_Even, J9 Conn_01x03, U1 BU33SD5WG-TR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

Commit message: Add files via upload
Changed lines of the file:
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@@
   (dimension (type aligned) (layer "Cmts.User")
     (pts (xy 24.96 21.07) (xy 34.995 21.07))
-    (height 0.215)
-    (gr_text "10,0350 mm" (at 29.9775 20.135) (layer "Cmts.User")
+    (height 0.223215)
+    (gr_text "10,0350 mm" (at 29.9775 20.143215) (layer "Cmts.User")
       (effects (font (size 1 1) (thickness 0.15)))
     )
@@
   (segment (start 140.19 68.41) (end 139.46 69.14) (width 0.2) (layer "B.Cu") (net 62))
   (segment (start 126.664823 69.024823) (end 126.34 68.7) (width 0.2) (layer "B.Cu") (net 62))
-  (segment (start 114.02295 99.55705) (end 89.8 99.55705) (width 0.2) (layer "F.Cu") (net 64))
+  (segment (start 125.47 88.11) (end 115.05 98.53) (width 0.2) (layer "F.Cu") (net 64))
+  (segment (start 90.82705 98.53) (end 89.8 99.55705) (width 0.2) (layer "F.Cu") (net 64))
+  (segment (start 125.23 70.54) (end 125.47 70.78) (width 0.2) (layer "F.Cu") (net 64))
+  (segment (start 125.47 70.78) (end 125.47 88.11) (width 0.2) (layer "F.Cu") (net 64))
+  (segment (start 125.225 66.7) (end 124.254314 66.7) (width 0.2) (layer "F.Cu") (net 64))
+  (segment (start 124.254314 66.7) (end 123.46 67.494315) (width 0.2) (layer "F.Cu") (net 64))
   (segment (start 89.8 100.1775) (end 89.8 99.55705) (width 0.25) (layer "F.Cu") (net 64))
+  (segment (start 123.46 67.494315) (end 123.46 68.768516) (width 0.2) (layer "F.Cu") (net 64))
+  (segment (start 115.05 98.53) (end 90.82705 98.53) (width 0.2) (layer "F.Cu") (net 64))
+  (segment (start 125.23 70.538516) (end 125.23 70.54) (width 0.2) (layer "F.Cu") (net 64))
   (segment (start 123.46 68.768516) (end 125.23 70.538516) (width 0.2) (layer "F.Cu") (net 64))
-  (segment (start 125.47 70.78) (end 125.47 88.11) (width 0.2) (layer "F.Cu") (net 64))
-  (segment (start 124.254314 66.7) (end 123.46 67.494315) (width 0.2) (layer "F.Cu") (net 64))
-  (segment (start 125.23 70.538516) (end 125.23 70.54) (width 0.2) (layer "F.Cu") (net 64))
-  (segment (start 123.46 67.494315) (end 123.46 68.768516) (width 0.2) (layer "F.Cu") (net 64))
-  (segment (start 125.225 66.7) (end 124.254314 66.7) (width 0.2) (layer "F.Cu") (net 64))
-  (segment (start 125.47 88.11) (end 114.02295 99.55705) (width 0.2) (layer "F.Cu") (net 64))
-  (segment (start 125.23 70.54) (end 125.47 70.78) (width 0.2) (layer "F.Cu") (net 64))
   (segment (start 137.95 66.1) (end 139.32 66.1) (width 0.25) (layer "F.Cu") (net 77))
   (segment (start 125.225 56.7) (end 126.32 56.7) (width 0.25) (layer "F.Cu") (net 77))
