File: Electronic Board/EC.kicad_sch (KiCad schematic)
At the start: 82 parts, among them J1 NMJ4HCD2, J2 4840.2201, J3 173950578, J4 NMJ4HCD2, J5 NMJ4HCD2, J6 NMJ4HCD2, SW2 SW_SPDT, U2 BU18SD2MG-MTR, U4 SGTL5000XNAA3, U5 IS42S16400J-xC, U502 BU33SD5WG-TR

Commit message: Add files via upload
Parts:
- D2, D502: footprint LED_SMD:LED_0201_0603Metric_Pad0.64x0.40mm_HandSolder -> LED_SMD:LED_0402_1005Metric_Pad0.77x0.64mm_HandSolder
- TP1, TP10, TP11, TP12, TP13, TP14, TP15, TP16, TP17, TP18, TP19, TP2, TP20, TP21, TP22, TP23, TP24, TP25, TP3, TP4, TP5, TP6, TP7, TP8, TP9: footprint TestPoint:TestPoint_Pad_D1.5mm -> Connector_Pin:Pin_D1.1mm_L8.5mm_W2.5mm_FlatFork
Other:
- note added: "SGTL5000 Audio Codec"
- note removed: "SGTL5000"
Changed lines of the file:
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@@
     (effects (font (size 1.27 1.27)) (justify left bottom))
   )
-  (text "SGTL5000\n\n\n \n" (at 52.07 85.09 0)
+  (text "SGTL5000 Audio Codec\n\n\n\n \n" (at 24.13 80.01 0)
     (effects (font (size 1.27 1.27)) (justify left bottom))
   )
@@
       (effects (font (size 1.27 1.27)) (justify left) hide)
     )
-    (property "Footprint" "TestPoint:TestPoint_Pad_D1.5mm" (at 85.09 203.2 0)
+    (property "Footprint" "Connector_Pin:Pin_D1.1mm_L8.5mm_W2.5mm_FlatFork" (at 85.09 203.2 0)
       (effects (font (size 1.27 1.27)) hide)
     )
@@
       (effects (font (size 1.27 1.27)) (justify left) hide)
     )
-    (property "Footprint" "TestPoint:TestPoint_Pad_D1.5mm" (at 59.69 142.24 0)
+    (property "Footprint" "Connector_Pin:Pin_D1.1mm_L8.5mm_W2.5mm_FlatFork" (at 59.69 142.24 0)
       (effects (font (size 1.27 1.27)) hide)
     )
@@
       (effects (font (size 1.27 1.27)) (justify left) hide)
     )
-    (property "Footprint" "TestPoint:TestPoint_Pad_D1.5mm" (at 48.26 251.46 0)
+    (property "Footprint" "Connector_Pin:Pin_D1.1mm_L8.5mm_W2.5mm_FlatFork" (at 48.26 251.46 0)
       (effects (font (size 1.27 1.27)) hide)
     )
@@
       (effects (font (size 1.27 1.27)) (justify left) hide)
     )
-    (property "Footprint" "TestPoint:TestPoint_Pad_D1.5mm" (at 243.84 34.29 0)
+    (property "Footprint" "Connector_Pin:Pin_D1.1mm_L8.5mm_W2.5mm_FlatFork" (at 243.84 34.29 0)
       (effects (font (size 1.27 1.27)) hide)
     )
@@
       (effects (font (size 1.27 1.27)) (justify left) hide)
     )
-    (property "Footprint" "TestPoint:TestPoint_Pad_D1.5mm" (at 57.15 139.7 0)
+    (property "Footprint" "Connector_Pin:Pin_D1.1mm_L8.5mm_W2.5mm_FlatFork" (at 57.15 139.7 0)
       (effects (font (size 1.27 1.27)) hide)
     )
@@
       (effects (font (size 1.27 1.27)) (justify left) hide)
     )
-    (property "Footprint" "TestPoint:TestPoint_Pad_D1.5mm" (at 288.29 35.56 0)
+    (property "Footprint" "Connector_Pin:Pin_D1.1mm_L8.5mm_W2.5mm_FlatFork" (at 288.29 35.56 0)
       (effects (font (size 1.27 1.27)) hide)
     )
@@
       (effects (font (size 1.27 1.27)) (justify left) hide)
     )
-    (property "Footprint" "TestPoint:TestPoint_Pad_D1.5mm" (at 50.8 129.54 0)
+    (property "Footprint" "Connector_Pin:Pin_D1.1mm_L8.5mm_W2.5mm_FlatFork" (at 50.8 129.54 0)
       (effects (font (size 1.27 1.27)) hide)
     )
@@
       (effects (font (size 1.27 1.27)) (justify left) hide)
     )
-    (property "Footprint" "TestPoint:TestPoint_Pad_D1.5mm" (at 54.61 137.16 0)
+    (property "Footprint" "Connector_Pin:Pin_D1.1mm_L8.5mm_W2.5mm_FlatFork" (at 54.61 137.16 0)
       (effects (font (size 1.27 1.27)) hide)
     )
@@
       (effects (font (size 1.27 1.27)) (justify left) hide)
     )
-    (property "Footprint" "TestPoint:TestPoint_Pad_D1.5mm" (at 139.7 29.21 0)
+    (property "Footprint" "Connector_Pin:Pin_D1.1mm_L8.5mm_W2.5mm_FlatFork" (at 139.7 29.21 0)
       (effects (font (size 1.27 1.27)) hide)
     )
@@
       (effects (font (size 1.27 1.27)) (justify left) hide)
     )
-    (property "Footprint" "TestPoint:TestPoint_Pad_D1.5mm" (at 64.77 149.86 0)
+    (property "Footprint" "Connector_Pin:Pin_D1.1mm_L8.5mm_W2.5mm_FlatFork" (at 64.77 149.86 0)
       (effects (font (size 1.27 1.27)) hide)
     )
@@
       (effects (font (size 1.27 1.27)) (justify left) hide)
     )
-    (property "Footprint" "TestPoint:TestPoint_Pad_D1.5mm" (at 43.18 261.62 0)
+    (property "Footprint" "Connector_Pin:Pin_D1.1mm_L8.5mm_W2.5mm_FlatFork" (at 43.18 261.62 0)
       (effects (font (size 1.27 1.27)) hide)
     )
@@
       (effects (font (size 1.27 1.27)) (justify left) hide)
     )
-    (property "Footprint" "TestPoint:TestPoint_Pad_D1.5mm" (at 107.95 109.22 0)
+    (property "Footprint" "Connector_Pin:Pin_D1.1mm_L8.5mm_W2.5mm_FlatFork" (at 107.95 109.22 0)
       (effects (font (size 1.27 1.27)) hide)
     )
@@
       (effects (font (size 1.27 1.27)) (justify left) hide)
     )
-    (property "Footprint" "TestPoint:TestPoint_Pad_D1.5mm" (at 80.01 35.56 0)
+    (property "Footprint" "Connector_Pin:Pin_D1.1mm_L8.5mm_W2.5mm_FlatFork" (at 80.01 35.56 0)
       (effects (font (size 1.27 1.27)) hide)
     )
@@
       (effects (font (size 1.27 1.27)) (justify left) hide)
     )
-    (property "Footprint" "TestPoint:TestPoint_Pad_D1.5mm" (at 194.31 31.75 0)
+    (property "Footprint" "Connector_Pin:Pin_D1.1mm_L8.5mm_W2.5mm_FlatFork" (at 194.31 31.75 0)
       (effects (font (size 1.27 1.27)) hide)
     )
@@
       (effects (font (size 1.27 1.27)) (justify left) hide)
     )
-    (property "Footprint" "TestPoint:TestPoint_Pad_D1.5mm" (at 52.07 210.82 0)
+    (property "Footprint" "Connector_Pin:Pin_D1.1mm_L8.5mm_W2.5mm_FlatFork" (at 52.07 210.82 0)
       (effects (font (size 1.27 1.27)) hide)
     )
@@
       (effects (font (size 1.27 1.27)) (justify left) hide)
     )
-    (property "Footprint" "TestPoint:TestPoint_Pad_D1.5mm" (at 344.17 189.23 0)
+    (property "Footprint" "Connector_Pin:Pin_D1.1mm_L8.5mm_W2.5mm_FlatFork" (at 344.17 189.23 0)
       (effects (font (size 1.27 1.27)) hide)
     )
@@
       (effects (font (size 1.27 1.27)) (justify left) hide)
     )
-    (property "Footprint" "TestPoint:TestPoint_Pad_D1.5mm" (at 68.58 109.22 0)
+    (property "Footprint" "Connector_Pin:Pin_D1.1mm_L8.5mm_W2.5mm_FlatFork" (at 68.58 109.22 0)
       (effects (font (size 1.27 1.27)) hide)
     )
@@
       (effects (font (size 1.27 1.27)) (justify left) hide)
     )
-    (property "Footprint" "TestPoint:TestPoint_Pad_D1.5mm" (at 45.72 248.92 0)
+    (property "Footprint" "Connector_Pin:Pin_D1.1mm_L8.5mm_W2.5mm_FlatFork" (at 45.72 248.92 0)
       (effects (font (size 1.27 1.27)) hide)
     )
@@
       (effects (font (size 1.27 1.27)) (justify left) hide)
     )
-    (property "Footprint" "TestPoint:TestPoint_Pad_D1.5mm" (at 43.18 246.38 0)
+    (property "Footprint" "Connector_Pin:Pin_D1.1mm_L8.5mm_W2.5mm_FlatFork" (at 43.18 246.38 0)
       (effects (font (size 1.27 1.27)) hide)
     )
@@
       (effects (font (size 1.27 1.27)) (justify left) hide)
     )
-    (property "Footprint" "TestPoint:TestPoint_Pad_D1.5mm" (at 44.45 264.16 0)
+    (property "Footprint" "Connector_Pin:Pin_D1.1mm_L8.5mm_W2.5mm_FlatFork" (at 44.45 264.16 0)
       (effects (font (size 1.27 1.27)) hide)
     )
@@
       (effects (font (size 1.27 1.27)) (justify right))
     )
-    (property "Footprint" "LED_SMD:LED_0201_0603Metric_Pad0.64x0.40mm_HandSolder" (at 142.24 34.29 90)
+    (property "Footprint" "LED_SMD:LED_0402_1005Metric_Pad0.77x0.64mm_HandSolder" (at 142.24 34.29 90)
       (effects (font (size 1.27 1.27)) hide)
     )
@@
       (effects (font (size 1.27 1.27)) (justify left))
     )
-    (property "Footprint" "LED_SMD:LED_0201_0603Metric_Pad0.64x0.40mm_HandSolder" (at 344.17 180.34 0)
+    (property "Footprint" "LED_SMD:LED_0402_1005Metric_Pad0.77x0.64mm_HandSolder" (at 344.17 180.34 0)
       (effects (font (size 1.27 1.27)) hide)
     )
@@
       (effects (font (size 1.27 1.27)) (justify left) hide)
     )
-    (property "Footprint" "TestPoint:TestPoint_Pad_D1.5mm" (at 62.23 147.32 0)
+    (property "Footprint" "Connector_Pin:Pin_D1.1mm_L8.5mm_W2.5mm_FlatFork" (at 62.23 147.32 0)
       (effects (font (size 1.27 1.27)) hide)
     )
@@
       (effects (font (size 1.27 1.27)) (justify left) hide)
     )
-    (property "Footprint" "TestPoint:TestPoint_Pad_D1.5mm" (at 50.8 254 0)
+    (property "Footprint" "Connector_Pin:Pin_D1.1mm_L8.5mm_W2.5mm_FlatFork" (at 50.8 254 0)
       (effects (font (size 1.27 1.27)) hide)
     )
@@
       (effects (font (size 1.27 1.27)) (justify left) hide)
     )
-    (property "Footprint" "TestPoint:TestPoint_Pad_D1.5mm" (at 52.07 134.62 0)
+    (property "Footprint" "Connector_Pin:Pin_D1.1mm_L8.5mm_W2.5mm_FlatFork" (at 52.07 134.62 0)
       (effects (font (size 1.27 1.27)) hide)
     )
@@
       (effects (font (size 1.27 1.27)) (justify left) hide)
     )
-    (property "Footprint" "TestPoint:TestPoint_Pad_D1.5mm" (at 53.34 259.08 0)
+    (property "Footprint" "Connector_Pin:Pin_D1.1mm_L8.5mm_W2.5mm_FlatFork" (at 53.34 259.08 0)
       (effects (font (size 1.27 1.27)) hide)
     )
@@
       (effects (font (size 1.27 1.27)) (justify left) hide)
     )
-    (property "Footprint" "TestPoint:TestPoint_Pad_D1.5mm" (at 52.07 256.54 0)
+    (property "Footprint" "Connector_Pin:Pin_D1.1mm_L8.5mm_W2.5mm_FlatFork" (at 52.07 256.54 0)
       (effects (font (size 1.27 1.27)) hide)
     )

Commit message: Add files via upload
Parts:
- added J8: Conn_02x07_Odd_Even, Connector_PinHeader_1.27mm:PinHeader_2x07_P1.27mm_Vertical_SMD, symbol Connector_Generic:Conn_02x07_Odd_Even
Connections:
- net +3.3V: now also J8.3 (Pin_3)
- net GND: now also J8.11 (Pin_11), J8.5 (Pin_5), J8.7 (Pin_7)
- net stm32/NRST renamed NRST
- net NRST: now also J8.12 (Pin_12)
- new net SWCLK: J8.6 (Pin_6)
- new net SWDIO: J8.4 (Pin_4)
- new net SWO: J8.8 (Pin_8)
- new net USART2_RX: J8.13 (Pin_13)
- new net USART2_TX: J8.14 (Pin_14)
- no-connect marks 16 -> 20
Other:
- sheet stm32 ports: added USART2_RX, USART2_TX; removed none
- note added: "ST Connector"

Commit message: Add files via upload
Parts:
- removed C1: 100uF, Capacitor_SMD:C_0402_1005Metric_Pad0.74x0.62mm_HandSolder, symbol Device:C
- removed C10, C11, C12, C13, C14, C15, C16, C20, C321 (x3), C40, C41, C42, C43, C44, C45, C46, C47, C48, C49: 100nF, Capacitor_SMD:C_0402_1005Metric_Pad0.74x0.62mm_HandSolder, symbol Device:C_Small
- removed C2: 100µF, Capacitor_SMD:C_0402_1005Metric_Pad0.74x0.62mm_HandSolder, symbol Device:C
- removed C3, C4, C5, C6: 1uF, Capacitor_SMD:C_0402_1005Metric_Pad0.74x0.62mm_HandSolder, symbol Device:C_Small
- removed D2: LED, LED_SMD:LED_0402_1005Metric_Pad0.77x0.64mm_HandSolder, symbol Device:LED
- removed D502: RED, LED_SMD:LED_0402_1005Metric_Pad0.77x0.64mm_HandSolder, symbol Device:LED_Small
- removed J1, J4, J5, J6: NMJ4HCD2, Connector_Audio:Jack_6.35mm_Neutrik_NMJ4HCD2_Horizontal, symbol Connector_Audio:NMJ4HCD2
- removed J2: 4840.2201, Library:Regulator4840-2201, symbol REGULATEUR 5V:4840.2201
- removed J3: 173950578, Library:CONN3_950578_WRE_173950578, symbol Regulator 5V:173950578
- removed J8: Conn_02x07_Odd_Even, Connector_PinHeader_1.27mm:PinHeader_2x07_P1.27mm_Vertical_SMD, symbol Connector_Generic:Conn_02x07_Odd_Even
- removed R3: 510, Resistor_SMD:R_0201_0603Metric_Pad0.64x0.40mm_HandSolder, symbol Device:R
- removed R3: 330, Resistor_SMD:R_0201_0603Metric_Pad0.64x0.40mm_HandSolder, symbol Device:R
- removed R502: 1k, Resistor_SMD:R_0603_1608Metric, symbol Device:R_Small
- removed RV1, RV10, RV2, RV3, RV4, RV5, RV6, RV7, RV8, RV9: 100k, Library:Potentiometer_Alpha_RD901F-40-00D_Single_Vertical, symbol Device:R_Potentiometer
- removed SW2: SW_SPDT, Library:RS_Pro_SPDT_8466720, symbol Switch:SW_SPDT
- removed TP1, TP15, TP17, TP2, TP25, TP3, TP4, TP7: TestPoint, Connector_Pin:Pin_D1.1mm_L8.5mm_W2.5mm_FlatFork, symbol Connector:TestPoint
- removed U2: BU18SD2MG-MTR, Package_TO_SOT_SMD:SOT-23-5, symbol WITNS_ROHM:BU18SD2MG-MTR
- removed U4: SGTL5000XNAA3, Package_DFN_QFN:QFN-32-1EP_5x5mm_P0.5mm_EP3.6x3.6mm, symbol Audio:SGTL5000XNAA3
- removed U5: IS42S16400J-xC, Package_SO:TSOP-II-54_22.2x10.16mm_P0.8mm, symbol Memory_RAM:IS42S16400J-xC
- removed U502: BU33SD5WG-TR, Package_TO_SOT_SMD:SOT-23-5, symbol WITNS_ROHM:BU33SD5WG-TR
Connections:
- net Codec/WS_I2S: now reaches TP23.1
- net +5V renamed STM32/SDNWE
- net A0 renamed Codec/SD_I2S
- net CK_I2S renamed Codec/Ve_guitare_L
- net D0 renamed Codec/DOUT_I2S
- net DOUT_I2S renamed Codec/Vs_guitare_L
- net NBL0 renamed STM32/NBL1
- net SCL_I2C renamed STM32/SDCKE1
- net SDA_I2C renamed STM32/SDCLK
- net SDCKE1 renamed STM32/NBL0
- net SDNCAS renamed Codec/SDA_I2C
- net SDNE1 renamed STM32/SDNCAS
- net SDNRAS renamed Codec/SCL_I2C
- net SDNWE renamed Codec/SYS_MCLK
- net Ve_guitare_L renamed Codec/CK_I2S
- net Ve_guitare_R renamed STM32/SDNE1 
- net Vs_guitare_R renamed STM32/SDNRAS
- no-connect marks 20 -> 0
Other:
- sheet stm32 renamed STM32
- added sheet Codec (codec.kicad_sch)
- added sheet Jacks IO ; Connectors ; Switch (jacks_IO.kicad_sch)
- added sheet Power Supply (power_supply.kicad_sch)
- added sheet ram (ram.kicad_sch)
- sheet STM32 ports: added A[0..11], BA[0..1], D[0..15]; removed A0, A1, A10, A11, A2, A3, A4, A5, A6, A7, A8, A9, BA0, BA1, BOOT0, BOOT1, Buffer, D0, D1, D10, D11, D12, D13, D14, D15, D2, D3, D4, D5, D6, D7, D8, D9, NRST, OSC32_IN, OSC32_OUT, OSC_IN, OSC_OUT, P0, P1, P2, P3, P4, P5, P6, P7, P8, P9, SWCLK, SWDIO, SWO, USART2_RX, USART2_TX, VDD, VSS
- note removed: "Buffer Button"
- note removed: "Jack Connectors"
- note removed: "Power Section"
- note removed: "RAM"
- note removed: "SGTL5000 Audio Codec"
- note removed: "ST Connector"
- note removed: "STM32"
- note removed: "Switch Regulator"
- note removed: "audio effects potentiometers"
- moved on the sheet: H1, H2, H3, H4

Commit message: Add files via upload
Parts:
- added TP26, TP7: TestPoint, Connector_Pin:Pin_D1.1mm_L8.5mm_W2.5mm_FlatFork, symbol Connector:TestPoint
Connections:
- net Codec/Ve_guitare_R: now also TP26.1
- net Codec/Vs_guitare_R: now also TP7.1
Changed lines of the file:
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@@
   (junction (at 69.85 114.3) (diameter 0) (color 0 0 0 0)
   )
+  (junction (at 72.39 116.84) (diameter 0) (color 0 0 0 0)
+  )
   (junction (at 116.84 111.76) (diameter 0) (color 0 0 0 0)
   )
@@
   (junction (at 129.54 127) (diameter 0) (color 0 0 0 0)
   )
-  (wire (pts (xy 66.04 121.92) (xy 80.01 121.92))
+  (junction (at 77.47 121.92) (diameter 0) (color 0 0 0 0)
+  )
+  (wire (pts (xy 66.04 121.92) (xy 77.47 121.92))
     (stroke (width 0) (type default))
   )
@@
     (stroke (width 0) (type default))
   )
+  (wire (pts (xy 77.47 121.92) (xy 80.01 121.92))
+    (stroke (width 0) (type default))
+  )
   (wire (pts (xy 69.85 114.3) (xy 80.01 114.3))
     (stroke (width 0) (type default))
@@
     (stroke (width 0) (type default))
   )
+  (wire (pts (xy 72.39 116.84) (xy 80.01 116.84))
+    (stroke (width 0) (type default))
+  )
   (wire (pts (xy 238.76 30.48) (xy 234.95 30.48))
     (stroke (width 0) (type default))
@@
     (stroke (width 0) (type default))
   )
-  (wire (pts (xy 66.04 116.84) (xy 80.01 116.84))
+  (wire (pts (xy 66.04 116.84) (xy 72.39 116.84))
     (stroke (width 0) (type default))
   )
@@
     (stroke (width 0) (type default))
   )
+  (wire (pts (xy 77.47 110.49) (xy 77.47 121.92))
+    (stroke (width 0) (type default))
+  )
   (wire (pts (xy 116.84 111.76) (xy 132.08 111.76))
     (stroke (width 0) (type default))
@@
   )
   (wire (pts (xy 116.84 99.06) (xy 116.84 111.76))
+    (stroke (width 0) (type default))
+  )
+  (wire (pts (xy 72.39 110.49) (xy 72.39 116.84))
     (stroke (width 0) (type default))
   )
@@
     )
   )
+  (symbol (lib_id "Connector:TestPoint") (at 72.39 110.49 0) (unit 1)
+    (in_bom yes) (on_board yes) (dnp no)
+    (property "Reference" "TP26" (at 72.39 104.14 90)
+      (effects (font (size 1.27 1.27)))
+    )
+    (property "Value" "TestPoint" (at 74.93 108.4579 0)
+      (effects (font (size 1.27 1.27)) (justify left) hide)
+    )
+    (property "Footprint" "Connector_Pin:Pin_D1.1mm_L8.5mm_W2.5mm_FlatFork" (at 77.47 110.49 0)
+      (effects (font (size 1.27 1.27)) hide)
+    )
+    (property "Datasheet" "~" (at 77.47 110.49 0)
+      (effects (font (size 1.27 1.27)) hide)
+    )
+    (pin "1")
+    (instances
+      (project "EC"
+        (path "/253d96fc-e3e7-475c-97d3-54a32a6a1970"
+          (reference "TP26") (unit 1)
+        )
+        (path "/253d96fc-e3e7-475c-97d3-54a32a6a1970/5e9c3599-d329-4855-bade-f50d28c2bc5b"
+          (reference "TP5") (unit 1)
+        )
+      )
+      (project "test_SGTL5000"
+        (path "/ac48c67b-93af-4f94-918a-70ca90985cf2/0bf4b4e6-cfdc-49c3-a185-97035ce0c8f7"
+          (reference "TP502") (unit 1)
+        )
+      )
+    )
+  )
   (symbol (lib_id "Connector:TestPoint") (at 184.15 55.88 0) (unit 1)
     (in_bom yes) (on_board yes) (dnp no)
@@
         )
       )
+      (project "test_SGTL5000"
+        (path "/ac48c67b-93af-4f94-918a-70ca90985cf2/0bf4b4e6-cfdc-49c3-a185-97035ce0c8f7"
+          (reference "TP502") (unit 1)
+        )
+      )
+    )
+  )
+  (symbol (lib_id "Connector:TestPoint") (at 77.47 110.49 0) (unit 1)
+    (in_bom yes) (on_board yes) (dnp no)
+    (property "Reference" "TP7" (at 77.47 104.14 90)
+      (effects (font (size 1.27 1.27)))
+    )
+    (property "Value" "TestPoint" (at 80.01 108.4579 0)
+      (effects (font (size 1.27 1.27)) (justify left) hide)
+    )
+    (property "Footprint" "Connector_Pin:Pin_D1.1mm_L8.5mm_W2.5mm_FlatFork" (at 82.55 110.49 0)
+      (effects (font (size 1.27 1.27)) hide)
+    )
+    (property "Datasheet" "~" (at 82.55 110.49 0)
+      (effects (font (size 1.27 1.27)) hide)
+    )
+    (pin "1")
+    (instances
+      (project "EC"
+        (path "/253d96fc-e3e7-475c-97d3-54a32a6a1970"
+          (reference "TP7") (unit 1)
+        )
+        (path "/253d96fc-e3e7-475c-97d3-54a32a6a1970/5e9c3599-d329-4855-bade-f50d28c2bc5b"
+          (reference "TP6") (unit 1)
+        )
+      )
