File: Electronic Board/codec.kicad_sch (KiCad schematic)
At the start: 8 parts, among them U4 SGTL5000XNAA3

Commit message: Add files via upload
Parts:
- removed TP10, TP11: TestPoint, Connector_Pin:Pin_D1.1mm_L8.5mm_W2.5mm_FlatFork, symbol Connector:TestPoint
Changed lines of the file:
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@@
   (junction (at 154.94 135.89) (diameter 0) (color 0 0 0 0)
-  )
-  (junction (at 175.26 80.01) (diameter 0) (color 0 0 0 0)
-  )
-  (junction (at 135.89 80.01) (diameter 0) (color 0 0 0 0)
   )
   (no_connect (at 170.18 95.25))
@@
     (stroke (width 0) (type default))
   )
-  (wire (pts (xy 170.18 80.01) (xy 175.26 80.01))
+  (wire (pts (xy 170.18 80.01) (xy 177.8 80.01))
     (stroke (width 0) (type default))
   )
@@
     (stroke (width 0) (type default))
   )
-  (wire (pts (xy 175.26 80.01) (xy 177.8 80.01))
-    (stroke (width 0) (type default))
-  )
-  (wire (pts (xy 135.89 80.01) (xy 139.7 80.01))
+  (wire (pts (xy 133.35 80.01) (xy 139.7 80.01))
     (stroke (width 0) (type default))
   )
@@
     (stroke (width 0) (type default))
   )
-  (wire (pts (xy 133.35 80.01) (xy 135.89 80.01))
-    (stroke (width 0) (type default))
-  )
   (wire (pts (xy 152.4 52.07) (xy 152.4 53.34))
     (stroke (width 0) (type default))
@@
     (stroke (width 0) (type default))
   )
-  (text "SGTL5000 Audio Codec\n\n\n\n \n" (at 96.52 55.88 0)
+  (text "SGTL5000 Audio Codec\n\n\n\n \n" (at 88.9 46.99 0)
     (effects (font (size 1.27 1.27)) (justify left bottom))
   )
@@
         (path "/253d96fc-e3e7-475c-97d3-54a32a6a1970/d27a2827-74a7-4246-8a59-7e614adac561"
           (reference "#PWR068") (unit 1)
-        )
-      )
-    )
-  )
-  (symbol (lib_id "Connector:TestPoint") (at 135.89 80.01 0) (unit 1)
-    (in_bom yes) (on_board yes) (dnp no)
-    (property "Reference" "TP10" (at 135.89 74.93 0)
-      (effects (font (size 1.27 1.27)))
-    )
-    (property "Value" "TestPoint" (at 138.43 77.9779 0)
-      (effects (font (size 1.27 1.27)) (justify left) hide)
-    )
-    (property "Footprint" "Connector_Pin:Pin_D1.1mm_L8.5mm_W2.5mm_FlatFork" (at 140.97 80.01 0)
-      (effects (font (size 1.27 1.27)) hide)
-    )
-    (property "Datasheet" "~" (at 140.97 80.01 0)
-      (effects (font (size 1.27 1.27)) hide)
-    )
-    (pin "1")
-    (instances
-      (project "EC"
-        (path "/253d96fc-e3e7-475c-97d3-54a32a6a1970"
-          (reference "TP10") (unit 1)
-        )
-        (path "/253d96fc-e3e7-475c-97d3-54a32a6a1970/d27a2827-74a7-4246-8a59-7e614adac561"
-          (reference "TP34") (unit 1)
-        )
-      )
-      (project "test_SGTL5000"
-        (path "/ac48c67b-93af-4f94-918a-70ca90985cf2/0bf4b4e6-cfdc-49c3-a185-97035ce0c8f7"
-          (reference "TP502") (unit 1)
         )
       )
@@
         )
       )
-    )
-  )
-  (symbol (lib_id "Connector:TestPoint") (at 175.26 80.01 0) (unit 1)
-    (in_bom yes) (on_board yes) (dnp no)
-    (property "Reference" "TP11" (at 175.26 74.93 0)
-      (effects (font (size 1.27 1.27)))
-    )
-    (property "Value" "TestPoint" (at 177.8 77.9779 0)
-      (effects (font (size 1.27 1.27)) (justify left) hide)
-    )
-    (property "Footprint" "Connector_Pin:Pin_D1.1mm_L8.5mm_W2.5mm_FlatFork" (at 180.34 80.01 0)
-      (effects (font (size 1.27 1.27)) hide)
-    )
-    (property "Datasheet" "~" (at 180.34 80.01 0)
-      (effects (font (size 1.27 1.27)) hide)
-    )
-    (pin "1")
-    (instances
-      (project "EC"
-        (path "/253d96fc-e3e7-475c-97d3-54a32a6a1970"
-          (reference "TP11") (unit 1)
-        )
-        (path "/253d96fc-e3e7-475c-97d3-54a32a6a1970/d27a2827-74a7-4246-8a59-7e614adac561"
-          (reference "TP35") (unit 1)
-        )
-      )
-      (project "test_SGTL5000"
-        (path "/ac48c67b-93af-4f94-918a-70ca90985cf2/0bf4b4e6-cfdc-49c3-a185-97035ce0c8f7"
-          (reference "TP502") (unit 1)
-        )
-      )
