File: Electronic Board/power_supply.kicad_sch (KiCad schematic)
At the start: 21 parts, among them J2 4840.2201, J3 173950578, U1 BU33SD5WG-TR, U2 BU33SD5WG-TR, U3 BU18SD2MG-MTR

Commit message: Add files via upload
Other:
- note added: "BU18SD2MG DANS LA BOITE"
Changed lines of the file:
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@@
+    (effects (font (size 1.27 1.27)) (justify left bottom))
+  )
+  (text "BU18SD2MG DANS LA BOITE\n" (at 106.68 128.27 0)
     (effects (font (size 1.27 1.27)) (justify left bottom))
   )

Commit message: Add files via upload
Parts:
- J2: value 4840.2201 -> 4840.2201 power connector
Other:
- note added: "C1 aluminium electrolyk capa"
- note removed: "C1 aluminium electrolyk capa 100µF/50V"
Changed lines of the file:
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@@
     (effects (font (size 1.27 1.27)) (justify left bottom))
   )
-  (text "C2 ceramic chip " (at 191.77 44.45 0)
+  (text "C2 ceramic chip " (at 187.96 40.64 0)
     (effects (font (size 1.27 1.27)) (justify left bottom))
   )
-  (text "C1 aluminium electrolyk capa 100µF/50V" (at 111.76 44.45 0)
+  (text "C1 aluminium electrolyk capa \n" (at 124.46 41.91 0)
     (effects (font (size 1.27 1.27)) (justify left bottom))
   )
-  (text "Pas les bonnes empreintes pour C1 et C2" (at 167.64 60.96 0)
+  (text "Pas les bonnes empreintes pour C1 et C2" (at 161.29 54.61 0)
     (effects (font (size 1.27 1.27)) (justify left bottom))
   )
@@
       (effects (font (size 1.524 1.524)))
     )
-    (property "Value" "4840.2201" (at 41.91 52.07 0)
+    (property "Value" "4840.2201 power connector " (at 46.99 26.67 0)
       (effects (font (size 1.524 1.524)))
     )
