File: Electronic Board/stm32.kicad_sch (KiCad schematic)
At the start: 14 parts, among them U6 STM32F446ZCTx

Commit message: Add files via upload
Parts:
- C304: value 1uF -> 100nF
Connections:
- net Buffer: now reaches U6.112 (PC11)
- no-connect marks 54 -> 53
Changed lines of the file:
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@@
   (no_connect (at 168.91 179.07))
   (no_connect (at 168.91 90.17))
-  (no_connect (at 229.87 171.45))
   (no_connect (at 229.87 196.85))
   (no_connect (at 168.91 97.79))
@@
     (stroke (width 0) (type default))
   )
+  (hierarchical_label "Buffer" (shape input) (at 229.87 171.45 0) (fields_autoplaced)
+    (effects (font (size 1.27 1.27)) (justify left))
+  )
   (hierarchical_label "A1" (shape input) (at 168.91 128.27 180) (fields_autoplaced)
     (effects (font (size 1.27 1.27)) (justify right))
@@
       (effects (font (size 1.27 1.27)) (justify right))
     )
-    (property "Value" "1uF" (at 232.41 38.1 90)
+    (property "Value" "100nF" (at 232.41 38.1 90)
       (effects (font (size 1.27 1.27)) (justify right))
     )
@@
       (effects (font (size 1.27 1.27)) (justify right))
     )
-    (property "Value" "1uF" (at 240.03 38.1 90)
+    (property "Value" "100nF" (at 240.03 38.1 90)
       (effects (font (size 1.27 1.27)) (justify right))
     )
@@
       (effects (font (size 1.27 1.27)) (justify right))
     )
-    (property "Value" "1uF" (at 220.98 38.1 90)
+    (property "Value" "100nF" (at 220.98 38.1 90)
       (effects (font (size 1.27 1.27)) (justify right))
     )
@@
       (effects (font (size 1.27 1.27)) (justify right))
     )
-    (property "Value" "1uF" (at 217.17 38.1 90)
+    (property "Value" "100nF" (at 217.17 38.1 90)
       (effects (font (size 1.27 1.27)) (justify right))
     )
@@
       (effects (font (size 1.27 1.27)) (justify right))
     )
-    (property "Value" "1uF" (at 247.65 38.1 90)
+    (property "Value" "100nF" (at 247.65 38.1 90)
       (effects (font (size 1.27 1.27)) (justify right))
     )
@@
       (effects (font (size 1.27 1.27)) (justify right))
     )
-    (property "Value" "1uF" (at 255.27 38.1 90)
+    (property "Value" "100nF" (at 255.27 38.1 90)
       (effects (font (size 1.27 1.27)) (justify right))
     )
@@
       (effects (font (size 1.27 1.27)) (justify right))
     )
-    (property "Value" "1uF" (at 259.08 38.1 90)
+    (property "Value" "100nF" (at 259.08 38.1 90)
       (effects (font (size 1.27 1.27)) (justify right))
     )
@@
       (effects (font (size 1.27 1.27)) (justify right))
     )
-    (property "Value" "1uF" (at 213.36 38.1 90)
+    (property "Value" "100nF" (at 213.36 38.1 90)
       (effects (font (size 1.27 1.27)) (justify right))
     )
@@
       (effects (font (size 1.27 1.27)) (justify right))
     )
-    (property "Value" "1uF" (at 243.84 38.1 90)
+    (property "Value" "100nF" (at 243.84 38.1 90)
       (effects (font (size 1.27 1.27)) (justify right))
     )
@@
       (effects (font (size 1.27 1.27)) (justify right))
     )
-    (property "Value" "1uF" (at 228.6 38.1 90)
+    (property "Value" "100nF" (at 228.6 38.1 90)
       (effects (font (size 1.27 1.27)) (justify right))
     )
@@
       (effects (font (size 1.27 1.27)) (justify right))
     )
-    (property "Value" "1uF" (at 236.22 38.1 90)
+    (property "Value" "100nF" (at 236.22 38.1 90)
       (effects (font (size 1.27 1.27)) (justify right))
     )
@@
       (effects (font (size 1.27 1.27)) (justify right))
     )
-    (property "Value" "1uF" (at 251.46 38.1 90)
+    (property "Value" "100nF" (at 251.46 38.1 90)
       (effects (font (size 1.27 1.27)) (justify right))
     )
@@
       (effects (font (size 1.27 1.27)) (justify right))
     )
-    (property "Value" "1uF" (at 224.79 38.1 90)
-      (effects (font (size 1.27 1.27)) (justify right))
-    )
+    (property "Value" "100nF" (at 224.79 38.1 90)
+      (effects (font (size 1.27 1.27)) (justify right))
+    )

Commit message: Add files via upload
Parts:
- C304: footprint Capacitor_SMD:C_0201_0603Metric_Pad0.64x0.40mm_HandSolder -> Capacitor_SMD:C_0402_1005Metric_Pad0.74x0.62mm_HandSolder
- C304: footprint Capacitor_SMD:C_0603_1608Metric -> Capacitor_SMD:C_0402_1005Metric_Pad0.74x0.62mm_HandSolder
Changed lines of the file:
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@@
       (effects (font (size 1.27 1.27)) (justify right))
     )
-    (property "Footprint" "Capacitor_SMD:C_0201_0603Metric_Pad0.64x0.40mm_HandSolder" (at 231.14 36.83 0)
+    (property "Footprint" "Capacitor_SMD:C_0402_1005Metric_Pad0.74x0.62mm_HandSolder" (at 231.14 36.83 0)
       (effects (font (size 1.27 1.27)) hide)
     )
@@
         )
       )
-      (project "TEST"
+      (project "EC"
         (path "/253d96fc-e3e7-475c-97d3-54a32a6a1970/562c3ef4-3faf-4a2b-b183-c065b2c5f1b8"
           (reference "C26") (unit 1)
@@
       (effects (font (size 1.27 1.27)) (justify right))
     )
-    (property "Footprint" "Capacitor_SMD:C_0603_1608Metric" (at 238.76 36.83 0)
+    (property "Footprint" "Capacitor_SMD:C_0402_1005Metric_Pad0.74x0.62mm_HandSolder" (at 238.76 36.83 0)
       (effects (font (size 1.27 1.27)) hide)
     )
@@
         )
       )
-      (project "TEST"
+      (project "EC"
         (path "/253d96fc-e3e7-475c-97d3-54a32a6a1970/562c3ef4-3faf-4a2b-b183-c065b2c5f1b8"
           (reference "C28") (unit 1)
@@
       (effects (font (size 1.27 1.27)) (justify right))
     )
-    (property "Footprint" "Capacitor_SMD:C_0201_0603Metric_Pad0.64x0.40mm_HandSolder" (at 219.71 36.83 0)
+    (property "Footprint" "Capacitor_SMD:C_0402_1005Metric_Pad0.74x0.62mm_HandSolder" (at 219.71 36.83 0)
       (effects (font (size 1.27 1.27)) hide)
     )
@@
         )
       )
-      (project "TEST"
+      (project "EC"
         (path "/253d96fc-e3e7-475c-97d3-54a32a6a1970/562c3ef4-3faf-4a2b-b183-c065b2c5f1b8"
           (reference "C23") (unit 1)
@@
       (effects (font (size 1.27 1.27)) (justify right))
     )
-    (property "Footprint" "Capacitor_SMD:C_0201_0603Metric_Pad0.64x0.40mm_HandSolder" (at 215.9 36.83 0)
+    (property "Footprint" "Capacitor_SMD:C_0402_1005Metric_Pad0.74x0.62mm_HandSolder" (at 215.9 36.83 0)
       (effects (font (size 1.27 1.27)) hide)
     )
@@
         )
       )
-      (project "TEST"
+      (project "EC"
         (path "/253d96fc-e3e7-475c-97d3-54a32a6a1970/562c3ef4-3faf-4a2b-b183-c065b2c5f1b8"
           (reference "C22") (unit 1)
@@
       (effects (font (size 1.27 1.27)) (justify right))
     )
-    (property "Footprint" "Capacitor_SMD:C_0201_0603Metric_Pad0.64x0.40mm_HandSolder" (at 246.38 36.83 0)
+    (property "Footprint" "Capacitor_SMD:C_0402_1005Metric_Pad0.74x0.62mm_HandSolder" (at 246.38 36.83 0)
       (effects (font (size 1.27 1.27)) hide)
     )
@@
         )
       )
-      (project "TEST"
+      (project "EC"
         (path "/253d96fc-e3e7-475c-97d3-54a32a6a1970/562c3ef4-3faf-4a2b-b183-c065b2c5f1b8"
           (reference "C30") (unit 1)
@@
       (effects (font (size 1.27 1.27)) (justify right))
     )
-    (property "Footprint" "Capacitor_SMD:C_0201_0603Metric_Pad0.64x0.40mm_HandSolder" (at 254 36.83 0)
+    (property "Footprint" "Capacitor_SMD:C_0402_1005Metric_Pad0.74x0.62mm_HandSolder" (at 254 36.83 0)
       (effects (font (size 1.27 1.27)) hide)
     )
@@
         )
       )
-      (project "TEST"
+      (project "EC"
         (path "/253d96fc-e3e7-475c-97d3-54a32a6a1970/562c3ef4-3faf-4a2b-b183-c065b2c5f1b8"
           (reference "C32") (unit 1)
@@
       (effects (font (size 1.27 1.27)) (justify right))
     )
-    (property "Footprint" "Capacitor_SMD:C_0201_0603Metric_Pad0.64x0.40mm_HandSolder" (at 257.81 36.83 0)
+    (property "Footprint" "Capacitor_SMD:C_0402_1005Metric_Pad0.74x0.62mm_HandSolder" (at 257.81 36.83 0)
       (effects (font (size 1.27 1.27)) hide)
     )
@@
         )
       )
-      (project "TEST"
+      (project "EC"
         (path "/253d96fc-e3e7-475c-97d3-54a32a6a1970/562c3ef4-3faf-4a2b-b183-c065b2c5f1b8"
           (reference "C33") (unit 1)
@@
     (pin "1")
     (instances
-      (project "TEST"
+      (project "EC"
         (path "/253d96fc-e3e7-475c-97d3-54a32a6a1970/562c3ef4-3faf-4a2b-b183-c065b2c5f1b8"
           (reference "#PWR021") (unit 1)
@@
       (effects (font (size 1.27 1.27)) (justify right))
     )
-    (property "Footprint" "Capacitor_SMD:C_0201_0603Metric_Pad0.64x0.40mm_HandSolder" (at 212.09 36.83 0)
+    (property "Footprint" "Capacitor_SMD:C_0402_1005Metric_Pad0.74x0.62mm_HandSolder" (at 212.09 36.83 0)
       (effects (font (size 1.27 1.27)) hide)
     )
@@
         )
       )
-      (project "TEST"
+      (project "EC"
         (path "/253d96fc-e3e7-475c-97d3-54a32a6a1970/562c3ef4-3faf-4a2b-b183-c065b2c5f1b8"
           (reference "C21") (unit 1)
@@
       (effects (font (size 1.27 1.27)) (justify right))
     )
-    (property "Footprint" "Capacitor_SMD:C_0201_0603Metric_Pad0.64x0.40mm_HandSolder" (at 242.57 36.83 0)
+    (property "Footprint" "Capacitor_SMD:C_0402_1005Metric_Pad0.74x0.62mm_HandSolder" (at 242.57 36.83 0)
       (effects (font (size 1.27 1.27)) hide)
     )
@@
         )
       )
-      (project "TEST"
+      (project "EC"
         (path "/253d96fc-e3e7-475c-97d3-54a32a6a1970/562c3ef4-3faf-4a2b-b183-c065b2c5f1b8"
           (reference "C29") (unit 1)
@@
       (effects (font (size 1.27 1.27)) (justify right))
     )
-    (property "Footprint" "Capacitor_SMD:C_0201_0603Metric_Pad0.64x0.40mm_HandSolder" (at 227.33 36.83 0)
+    (property "Footprint" "Capacitor_SMD:C_0402_1005Metric_Pad0.74x0.62mm_HandSolder" (at 227.33 36.83 0)
       (effects (font (size 1.27 1.27)) hide)
     )
@@
         )
       )
-      (project "TEST"
+      (project "EC"
         (path "/253d96fc-e3e7-475c-97d3-54a32a6a1970/562c3ef4-3faf-4a2b-b183-c065b2c5f1b8"
           (reference "C25") (unit 1)
@@
       (effects (font (size 1.27 1.27)) (justify right))
     )
-    (property "Footprint" "Capacitor_SMD:C_0201_0603Metric_Pad0.64x0.40mm_HandSolder" (at 234.95 36.83 0)
+    (property "Footprint" "Capacitor_SMD:C_0402_1005Metric_Pad0.74x0.62mm_HandSolder" (at 234.95 36.83 0)
       (effects (font (size 1.27 1.27)) hide)
     )
@@
         )
       )
-      (project "TEST"
+      (project "EC"
         (path "/253d96fc-e3e7-475c-97d3-54a32a6a1970/562c3ef4-3faf-4a2b-b183-c065b2c5f1b8"
           (reference "C27") (unit 1)
@@
       (effects (font (size 1.27 1.27)) (justify right))
     )
-    (property "Footprint" "Capacitor_SMD:C_0201_0603Metric_Pad0.64x0.40mm_HandSolder" (at 250.19 36.83 0)
+    (property "Footprint" "Capacitor_SMD:C_0402_1005Metric_Pad0.74x0.62mm_HandSolder" (at 250.19 36.83 0)
       (effects (font (size 1.27 1.27)) hide)
     )
@@
         )
       )
-      (project "TEST"
+      (project "EC"
         (path "/253d96fc-e3e7-475c-97d3-54a32a6a1970/562c3ef4-3faf-4a2b-b183-c065b2c5f1b8"
           (reference "C31") (unit 1)
@@
       (effects (font (size 1.27 1.27)) (justify right))
     )
-    (property "Footprint" "Capacitor_SMD:C_0201_0603Metric_Pad0.64x0.40mm_HandSolder" (at 223.52 36.83 0)
+    (property "Footprint" "Capacitor_SMD:C_0402_1005Metric_Pad0.74x0.62mm_HandSolder" (at 223.52 36.83 0)
       (effects (font (size 1.27 1.27)) hide)
     )
@@
         )
       )
-      (project "TEST"
+      (project "EC"
         (path "/253d96fc-e3e7-475c-97d3-54a32a6a1970/562c3ef4-3faf-4a2b-b183-c065b2c5f1b8"
           (reference "C24") (unit 1)
@@
     (pin "99")
     (instances
-      (project "TEST"
+      (project "EC"
         (path "/253d96fc-e3e7-475c-97d3-54a32a6a1970"
           (reference "U6") (unit 1)

Commit message: Add files via upload
Parts:
- added C304: 4.7u, Capacitor_SMD:C_0603_1608Metric, symbol Device:C_Small
Connections:
- net GND: now also C304.2
- net VDD: now also C304.1
- net USART2_TX: now reaches U6.36 (PA2)
- net USART2_RX: now reaches U6.37 (PA3)
- no-connect marks 53 -> 51
Changed lines of the file:
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@@
   (junction (at 186.69 44.45) (diameter 0) (color 0 0 0 0)
   )
+  (junction (at 257.81 34.29) (diameter 0) (color 0 0 0 0)
+  )
   (junction (at 250.19 39.37) (diameter 0) (color 0 0 0 0)
   )
@@
   (junction (at 250.19 34.29) (diameter 0) (color 0 0 0 0)
   )
+  (junction (at 254 39.37) (diameter 0) (color 0 0 0 0)
+  )
   (junction (at 219.71 39.37) (diameter 0) (color 0 0 0 0)
   )
   (junction (at 254 34.29) (diameter 0) (color 0 0 0 0)
   )
-  (junction (at 254 39.37) (diameter 0) (color 0 0 0 0)
-  )
   (junction (at 246.38 34.29) (diameter 0) (color 0 0 0 0)
   )
@@
   )
   (junction (at 227.33 34.29) (diameter 0) (color 0 0 0 0)
+  )
+  (junction (at 257.81 39.37) (diameter 0) (color 0 0 0 0)
   )
   (junction (at 214.63 44.45) (diameter 0) (color 0 0 0 0)
@@
   (no_connect (at 168.91 69.85))
   (no_connect (at 229.87 217.17))
-  (no_connect (at 229.87 64.77))
   (no_connect (at 229.87 201.93))
   (no_connect (at 168.91 110.49))
@@
   (no_connect (at 168.91 146.05))
   (no_connect (at 168.91 143.51))
-  (no_connect (at 229.87 62.23))
   (no_connect (at 229.87 85.09))
   (no_connect (at 229.87 67.31))
@@
     (stroke (width 0) (type default))
   )
+  (wire (pts (xy 257.81 34.29) (xy 261.62 34.29))
+    (stroke (width 0) (type default))
+  )
   (wire (pts (xy 207.01 44.45) (xy 209.55 44.45))
     (stroke (width 0) (type default))
@@
     (stroke (width 0) (type default))
   )
+  (wire (pts (xy 257.81 39.37) (xy 261.62 39.37))
+    (stroke (width 0) (type default))
+  )
   (wire (pts (xy 223.52 34.29) (xy 227.33 34.29))
     (stroke (width 0) (type default))
@@
     (stroke (width 0) (type default))
   )
+  (wire (pts (xy 223.52 39.37) (xy 227.33 39.37))
+    (stroke (width 0) (type default))
+  )
+  (wire (pts (xy 200.66 234.95) (xy 200.66 237.49))
+    (stroke (width 0) (type default))
+  )
+  (wire (pts (xy 207.01 44.45) (xy 207.01 49.53))
+    (stroke (width 0) (type default))
+  )
+  (wire (pts (xy 231.14 34.29) (xy 234.95 34.29))
+    (stroke (width 0) (type default))
+  )
+  (wire (pts (xy 227.33 39.37) (xy 231.14 39.37))
+    (stroke (width 0) (type default))
+  )
+  (wire (pts (xy 201.93 44.45) (xy 204.47 44.45))
+    (stroke (width 0) (type default))
+  )
+  (wire (pts (xy 184.15 44.45) (xy 186.69 44.45))
+    (stroke (width 0) (type default))
+  )
+  (wire (pts (xy 189.23 44.45) (xy 191.77 44.45))
+    (stroke (width 0) (type default))
+  )
+  (wire (pts (xy 191.77 44.45) (xy 191.77 49.53))
+    (stroke (width 0) (type default))
+  )
+  (wire (pts (xy 215.9 34.29) (xy 219.71 34.29))
+    (stroke (width 0) (type default))
+  )
+  (wire (pts (xy 199.39 34.29) (xy 199.39 44.45))
+    (stroke (width 0) (type default))
+  )
+  (wire (pts (xy 219.71 34.29) (xy 223.52 34.29))
+    (stroke (width 0) (type default))
+  )
+  (wire (pts (xy 194.31 44.45) (xy 196.85 44.45))
+    (stroke (width 0) (type default))
+  )
+  (wire (pts (xy 234.95 34.29) (xy 238.76 34.29))
+    (stroke (width 0) (type default))
+  )
+  (wire (pts (xy 209.55 44.45) (xy 209.55 49.53))
+    (stroke (width 0) (type default))
+  )
+  (wire (pts (xy 246.38 39.37) (xy 250.19 39.37))
+    (stroke (width 0) (type default))
+  )
+  (wire (pts (xy 231.14 39.37) (xy 234.95 39.37))
+    (stroke (width 0) (type default))
+  )
+  (wire (pts (xy 254 34.29) (xy 257.81 34.29))
+    (stroke (width 0) (type default))
+  )
+  (wire (pts (xy 238.76 39.37) (xy 242.57 39.37))
+    (stroke (width 0) (type default))
+  )
+  (wire (pts (xy 212.09 39.37) (xy 212.09 40.64))
+    (stroke (width 0) (type default))
+  )
   (wire (pts (xy 254 39.37) (xy 257.81 39.37))
     (stroke (width 0) (type default))
   )
-  (wire (pts (xy 223.52 39.37) (xy 227.33 39.37))
-    (stroke (width 0) (type default))
-  )
-  (wire (pts (xy 200.66 234.95) (xy 200.66 237.49))
-    (stroke (width 0) (type default))
-  )
-  (wire (pts (xy 207.01 44.45) (xy 207.01 49.53))
-    (stroke (width 0) (type default))
-  )
-  (wire (pts (xy 231.14 34.29) (xy 234.95 34.29))
-    (stroke (width 0) (type default))
-  )
-  (wire (pts (xy 227.33 39.37) (xy 231.14 39.37))
-    (stroke (width 0) (type default))
-  )
-  (wire (pts (xy 201.93 44.45) (xy 204.47 44.45))
-    (stroke (width 0) (type default))
-  )
-  (wire (pts (xy 184.15 44.45) (xy 186.69 44.45))
-    (stroke (width 0) (type default))
-  )
-  (wire (pts (xy 189.23 44.45) (xy 191.77 44.45))
-    (stroke (width 0) (type default))
-  )
-  (wire (pts (xy 191.77 44.45) (xy 191.77 49.53))
-    (stroke (width 0) (type default))
-  )
-  (wire (pts (xy 215.9 34.29) (xy 219.71 34.29))
-    (stroke (width 0) (type default))
-  )
-  (wire (pts (xy 199.39 34.29) (xy 199.39 44.45))
-    (stroke (width 0) (type default))
-  )
-  (wire (pts (xy 219.71 34.29) (xy 223.52 34.29))
-    (stroke (width 0) (type default))
-  )
-  (wire (pts (xy 194.31 44.45) (xy 196.85 44.45))
-    (stroke (width 0) (type default))
-  )
-  (wire (pts (xy 234.95 34.29) (xy 238.76 34.29))
-    (stroke (width 0) (type default))
-  )
-  (wire (pts (xy 209.55 44.45) (xy 209.55 49.53))
-    (stroke (width 0) (type default))
-  )
-  (wire (pts (xy 246.38 39.37) (xy 250.19 39.37))
-    (stroke (width 0) (type default))
-  )
-  (wire (pts (xy 231.14 39.37) (xy 234.95 39.37))
-    (stroke (width 0) (type default))
-  )
-  (wire (pts (xy 254 34.29) (xy 257.81 34.29))
-    (stroke (width 0) (type default))
-  )
-  (wire (pts (xy 238.76 39.37) (xy 242.57 39.37))
-    (stroke (width 0) (type default))
-  )
-  (wire (pts (xy 212.09 39.37) (xy 212.09 40.64))
-    (stroke (width 0) (type default))
-  )
   (wire (pts (xy 212.09 39.37) (xy 215.9 39.37))
     (stroke (width 0) (type default))
@@
     (effects (font (size 1.27 1.27)) (justify left))
   )
+  (hierarchical_label "USART2_RX" (shape input) (at 229.87 64.77 0) (fields_autoplaced)
+    (effects (font (size 1.27 1.27)) (justify left))
+  )
   (hierarchical_label "DOUT_I2C" (shape input) (at 229.87 123.19 0) (fields_autoplaced)
     (effects (font (size 1.27 1.27)) (justify left))
@@
   )
   (hierarchical_label "SYS_MCLK" (shape input) (at 229.87 59.69 0) (fields_autoplaced)
+    (effects (font (size 1.27 1.27)) (justify left))
+  )
+  (hierarchical_label "USART2_TX" (shape input) (at 229.87 62.23 0) (fields_autoplaced)
     (effects (font (size 1.27 1.27)) (justify left))
   )
@@
         )
       )
+      (project "audio_codec"
+        (path "/3540f935-04c6-4343-9dea-becd1b5c41b8"
+          (reference "C4") (unit 1)
+        )
+      )
+      (project "STM32F446_memory_demo1"
+        (path "/d10f480e-e97b-4ca7-9726-e760006f5bda/00b0349e-9bf6-4d86-8783-f8df71c96935"
+          (reference "C304") (unit 1)
+        )
+      )
+    )
+  )
+  (symbol (lib_id "Device:C_Small") (at 261.62 36.83 0) (mirror y) (unit 1)
+    (in_bom yes) (on_board yes) (dnp no)
+    (property "Reference" "C304" (at 262.89 31.115 90)
+      (effects (font (size 1.27 1.27)) (justify right))
+    )
+    (property "Value" "4.7u" (at 262.89 38.1 90)
+      (effects (font (size 1.27 1.27)) (justify right))
+    )
+    (property "Footprint" "Capacitor_SMD:C_0603_1608Metric" (at 261.62 36.83 0)
+      (effects (font (size 1.27 1.27)) hide)
+    )
+    (property "Datasheet" "~" (at 261.62 36.83 0)
+      (effects (font (size 1.27 1.27)) hide)
+    )
+    (pin "1")
+    (pin "2")
+    (instances
+      (project "stm32f446"
+        (path "/04477595-6581-45be-afcf-f7e974c5582c"
+          (reference "C304") (unit 1)
+        )
+      )
+      (project "EC"
+        (path "/253d96fc-e3e7-475c-97d3-54a32a6a1970/562c3ef4-3faf-4a2b-b183-c065b2c5f1b8"
+          (reference "C17") (unit 1)
+        )
+      )

Commit message: Add files via upload
Parts:
- added C20, C304 (x2), C40, C41, C42, C43, C44, C45, C46, C47, C48, C49: 100nF, Capacitor_SMD:C_0402_1005Metric_Pad0.74x0.62mm_HandSolder, symbol Device:C_Small
- added C304 (x2): 2.2uF, Capacitor_SMD:C_0402_1005Metric_Pad0.74x0.62mm_HandSolder, symbol Device:C_Small
- added D2: LED, LED_SMD:LED_0402_1005Metric_Pad0.77x0.64mm_HandSolder, symbol Device:LED
- added J8: Conn_02x07_Odd_Even, Connector_PinHeader_1.27mm:PinHeader_2x07_P1.27mm_Vertical_SMD, symbol Connector_Generic:Conn_02x07_Odd_Even
- added J9: Conn_01x03, Connector_JST:JST_XH_S3B-XH-A-1_1x03_P2.50mm_Horizontal, symbol Connector_Generic:Conn_01x03
- added R3: 330, Resistor_SMD:R_0201_0603Metric_Pad0.64x0.40mm_HandSolder, symbol Device:R
- added R6: 510, Resistor_SMD:R_0201_0603Metric_Pad0.64x0.40mm_HandSolder, symbol Device:R
- added RV1, RV10, RV2, RV3, RV4, RV5, RV6, RV7, RV8, RV9: 100k, Library:Potentiometer_Alpha_RD901F-40-00D_Single_Vertical, symbol Device:R_Potentiometer
Connections:
- net VSS is gone; now on net GND: U6.107 (VSS), U6.120 (VSS), U6.130 (VSS), U6.16 (VSS), U6.31 (VSSA), U6.38 (VSS), U6.51 (VSS), U6.61 (VSS), U6.83 (VSS), U6.94 (VSS)
- net GND: now also U6.32 (VREF+), C20.2, C304.2, C304.2, C304.2, C304.2, C40.2, C41.2, C42.2, C43.2, C44.2, C45.2, C46.2, C47.2, C48.2, C49.2, J8.11 (Pin_11), J8.5 (Pin_5), J8.7 (Pin_7), R6.1, RV1.3, RV10.3, RV2.3, RV3.3, RV4.3, RV5.3, RV6.3, RV7.3, RV8.3, RV9.3
- net NRST: now also C20.1, J8.12 (Pin_12)
- net SWCLK: now also J8.6 (Pin_6)
- net SWDIO: now also J8.4 (Pin_4)
- net SWO: now also J8.8 (Pin_8)
- net USART2_RX: now also J8.13 (Pin_13)
- net USART2_TX: now also J8.14 (Pin_14)
- net at U6.106 (VCAP_2): now also C304.1
- net +3.3V: now reaches U6.143 (PDR_ON)
- net +3.3V: now also C304.1, C304.1, C304.1, C304.1, C304.1, C304.1, C304.1, C304.1, C304.1, C304.1, C304.1, C304.1, C304.1, U6.108 (VDD), U6.121 (VDD), U6.131 (VDD), U6.144 (VDD), U6.17 (VDD), U6.30 (VDD), U6.39 (VDD), U6.52 (VDD), U6.6 (VBAT), U6.62 (VDD), U6.72 (VDD), U6.84 (VDD), U6.95 (VDDUSB), C304.1, C304.1, J8.3 (Pin_3), J9.1 (Pin_1), RV1.1, RV10.1, RV2.1, RV3.1, RV4.1, RV5.1, RV6.1, RV7.1, RV8.1, RV9.1
- net at U6.71 (VCAP_1): now also C304.1
- net BOOT0: no longer names the net of U6.138 (BOOT0)
- net BOOT0: now also R6.2
- net BOOT1: no longer names the net of U6.48 (PB2)
- net Buffer: no longer names the net of U6.112 (PC11)
- net Buffer: now also D2.1 (K)
- net OSC32_IN: no longer names the net of U6.8 (PC14)
- net OSC32_OUT: no longer names the net of U6.9 (PC15)
- net OSC_IN: no longer names the net of U6.23 (PH0)
- net OSC_OUT: no longer names the net of U6.24 (PH1)
- net P0 renamed Pot_0
- net Pot_0: now also C40.1, RV1.2
- net P1 renamed Pot_1
- net Pot_1: now also C43.1, RV4.2
- net P2 renamed Pot_2
- net Pot_2: now also C46.1, RV7.2
- net P3 renamed Pot_3
- net Pot_3: now also C49.1, RV10.2
- net P4 renamed Pot_4
- net Pot_4: now also C41.1, RV2.2
- net P5 renamed Pot_5
- net Pot_5: now also C44.1, RV5.2
- net P6 renamed Pot_6
- net Pot_6: now also C47.1, RV8.2
- net P7 renamed Pot_7
- net Pot_7: now also C45.1, RV6.2
- net P8: no longer names the net of U6.111 (PC10)
- net P8: no longer U6.46 (PB0)
- net P9 renamed Pot_9
- net Pot_9: now also C42.1, RV3.2
- removed net VDD: C304.1, C304.1, C304.1, C304.1, C304.1, C304.1, C304.1, C304.1, C304.1, C304.1, C304.1, C304.1, C304.1, C304.1, U6.108 (VDD), U6.121 (VDD), U6.131 (VDD), U6.144 (VDD), U6.17 (VDD), U6.30 (VDD), U6.33 (VDDA), U6.39 (VDD), U6.52 (VDD), U6.6 (VBAT), U6.62 (VDD), U6.72 (VDD), U6.84 (VDD), U6.95 (VDDUSB)
- new net: D2.2 (A), R3.1
- new net: J9.3 (Pin_3), R3.2
- new net +3.3VA: C304.1, U6.33 (VDDA)
- new net Pot_8: C48.1, RV9.2, U6.46 (PB0)
- no-connect marks 51 -> 58
Other:
- note added: "ST Connector"
- moved on the sheet: C304, U6
