File: Electronic Board/stm32.kicad_sch (KiCad schematic)
At the start: 45 parts, among them J8 Conn_02x07_Odd_Even, J9 Conn_01x03, U6 STM32F446ZCTx

Commit message: Add files via upload
Parts:
- added D2: LED, LED_SMD:LED_0402_1005Metric_Pad0.77x0.64mm_HandSolder, symbol Device:LED
- added J9: Conn_01x03, Connector_JST:JST_XH_S3B-XH-A-1_1x03_P2.50mm_Horizontal, symbol Connector_Generic:Conn_01x03
- added R3: 330, Resistor_SMD:R_0201_0603Metric_Pad0.64x0.40mm_HandSolder, symbol Device:R
Connections:
- net +3.3V: now also J9.1 (Pin_1)
- net at U6.113 (PC12): now also D2.1 (K)
- new net: D2.2 (A), R3.1
- new net: J9.3 (Pin_3), R3.2
Changed lines of the file:
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@@
   (no_connect (at 210.82 91.44))
   (no_connect (at 134.62 232.41))
+  (no_connect (at 173.99 201.93))
   (no_connect (at 134.62 207.01))
   (no_connect (at 73.66 87.63))
@@
   (no_connect (at 134.62 90.17))
   (no_connect (at 73.66 194.31))
-  (no_connect (at 134.62 186.69))
   (no_connect (at 73.66 113.03))
   (no_connect (at 210.82 81.28))
@@
     (stroke (width 0) (type default))
   )
+  (wire (pts (xy 151.13 208.28) (xy 143.51 208.28))
+    (stroke (width 0) (type default))
+  )
   (wire (pts (xy 68.58 91.44) (xy 68.58 82.55))
     (stroke (width 0) (type default))
@@
     (stroke (width 0) (type default))
   )
+  (wire (pts (xy 143.51 186.69) (xy 134.62 186.69))
+    (stroke (width 0) (type default))
+  )
   (bus (pts (xy 38.1 173.99) (xy 38.1 176.53))
     (stroke (width 0) (type default))
@@
     (stroke (width 0) (type default))
   )
+  (wire (pts (xy 168.91 204.47) (xy 173.99 204.47))
+    (stroke (width 0) (type default))
+  )
   (wire (pts (xy 34.29 213.36) (xy 35.56 213.36))
     (stroke (width 0) (type default))
@@
     (stroke (width 0) (type default))
   )
+  (wire (pts (xy 166.37 196.85) (xy 166.37 199.39))
+    (stroke (width 0) (type default))
+  )
   (bus (pts (xy 38.1 151.13) (xy 39.37 151.13))
     (stroke (width 0) (type default))
@@
     (stroke (width 0) (type default))
   )
+  (wire (pts (xy 173.99 199.39) (xy 166.37 199.39))
+    (stroke (width 0) (type default))
+  )
   (wire (pts (xy 124.46 38.1) (xy 128.27 38.1))
     (stroke (width 0) (type default))
@@
     (stroke (width 0) (type default))
   )
+  (wire (pts (xy 143.51 208.28) (xy 143.51 186.69))
+    (stroke (width 0) (type default))
+  )
   (wire (pts (xy 137.16 176.53) (xy 134.62 176.53))
     (stroke (width 0) (type default))
@@
     (stroke (width 0) (type default))
   )
+  (wire (pts (xy 168.91 208.28) (xy 168.91 204.47))
+    (stroke (width 0) (type default))
+  )
   (wire (pts (xy 73.66 224.79) (xy 62.23 224.79))
     (stroke (width 0) (type default))
@@
   )
   (bus (pts (xy 38.1 200.66) (xy 38.1 203.2))
+    (stroke (width 0) (type default))
+  )
+  (wire (pts (xy 158.75 208.28) (xy 161.29 208.28))
     (stroke (width 0) (type default))
   )
@@
     )
   )
+  (symbol (lib_id "Device:LED") (at 154.94 208.28 0) (mirror x) (unit 1)
+    (in_bom yes) (on_board yes) (dnp no)
+    (property "Reference" "D2" (at 152.7175 210.82 0)
+      (effects (font (size 1.27 1.27)) (justify left))
+    )
+    (property "Value" "LED" (at 151.13 213.36 0)
+      (effects (font (size 1.27 1.27)) (justify left))
+    )
+    (property "Footprint" "LED_SMD:LED_0402_1005Metric_Pad0.77x0.64mm_HandSolder" (at 154.94 208.28 0)
+      (effects (font (size 1.27 1.27)) hide)
+    )
+    (property "Datasheet" "~" (at 154.94 208.28 0)
+      (effects (font (size 1.27 1.27)) hide)
+    )
+    (pin "1")
+    (pin "2")
+    (instances
+      (project "EC"
+        (path "/253d96fc-e3e7-475c-97d3-54a32a6a1970"
+          (reference "D2") (unit 1)
+        )
+        (path "/253d96fc-e3e7-475c-97d3-54a32a6a1970/562c3ef4-3faf-4a2b-b183-c065b2c5f1b8"
+          (reference "D4") (unit 1)
+        )
+      )
+    )
+  )
   (symbol (lib_id "Device:R_Potentiometer") (at 313.69 226.06 0) (unit 1)
     (in_bom yes) (on_board yes) (dnp no)
@@
     )
   )
+  (symbol (lib_id "Device:R") (at 165.1 208.28 90) (mirror x) (unit 1)
+    (in_bom yes) (on_board yes) (dnp no)
+    (property "Reference" "R3" (at 167.64 211.455 90)
+      (effects (font (size 1.27 1.27)) (justify left))
+    )
+    (property "Value" "330" (at 167.64 213.995 90)
+      (effects (font (size 1.27 1.27)) (justify left))
+    )
+    (property "Footprint" "Resistor_SMD:R_0201_0603Metric_Pad0.64x0.40mm_HandSolder" (at 165.1 206.502 90)
+      (effects (font (size 1.27 1.27)) hide)
+    )
+    (property "Datasheet" "~" (at 165.1 208.28 0)
+      (effects (font (size 1.27 1.27)) hide)
+    )
+    (pin "1")
+    (pin "2")
+    (instances
+      (project "EC"
+        (path "/253d96fc-e3e7-475c-97d3-54a32a6a1970"
+          (reference "R3") (unit 1)
+        )
+        (path "/253d96fc-e3e7-475c-97d3-54a32a6a1970/562c3ef4-3faf-4a2b-b183-c065b2c5f1b8"
+          (reference "R4") (unit 1)
+        )
+      )
+    )
+  )
   (symbol (lib_id "power:GND") (at 50.8 80.01 0) (unit 1)
     (in_bom yes) (on_board yes) (dnp no)
@@
         (path "/253d96fc-e3e7-475c-97d3-54a32a6a1970/562c3ef4-3faf-4a2b-b183-c065b2c5f1b8"
           (reference "#PWR058") (unit 1)
+        )
+      )
+    )
+  )
+  (symbol (lib_id "power:+3.3V") (at 166.37 196.85 0) (mirror y) (unit 1)
+    (in_bom yes) (on_board yes) (dnp no) (fields_autoplaced)
+    (property "Reference" "#PWR027" (at 166.37 200.66 0)
+      (effects (font (size 1.27 1.27)) hide)
+    )
+    (property "Value" "+3.3V" (at 166.37 193.04 0)
+      (effects (font (size 1.27 1.27)))
+    )
+    (property "Footprint" "" (at 166.37 196.85 0)
+      (effects (font (size 1.27 1.27)) hide)
+    )
+    (property "Datasheet" "" (at 166.37 196.85 0)
+      (effects (font (size 1.27 1.27)) hide)
+    )
+    (pin "1")
+    (instances
+      (project "EC"
+        (path "/253d96fc-e3e7-475c-97d3-54a32a6a1970"
+          (reference "#PWR027") (unit 1)
+        )
+        (path "/253d96fc-e3e7-475c-97d3-54a32a6a1970/562c3ef4-3faf-4a2b-b183-c065b2c5f1b8"
+          (reference "#PWR061") (unit 1)
         )
       )
@@
         )
       )
+    )
+  )
+  (symbol (lib_id "Connector_Generic:Conn_01x03") (at 179.07 201.93 0) (unit 1)
+    (in_bom yes) (on_board yes) (dnp no)
+    (property "Reference" "J9" (at 181.61 201.295 0)
+      (effects (font (size 1.27 1.27)) (justify left))
+    )
+    (property "Value" "Conn_01x03" (at 175.26 196.85 0)
+      (effects (font (size 1.27 1.27)) (justify left))
+    )
+    (property "Footprint" "Connector_JST:JST_XH_S3B-XH-A-1_1x03_P2.50mm_Horizontal" (at 179.07 201.93 0)
+      (effects (font (size 1.27 1.27)) hide)
+    )
+    (property "Datasheet" "~" (at 179.07 201.93 0)
+      (effects (font (size 1.27 1.27)) hide)
+    )
+    (pin "1")
+    (pin "2")
+    (pin "3")
+    (instances
+      (project "EC"
+        (path "/253d96fc-e3e7-475c-97d3-54a32a6a1970"
+          (reference "J9") (unit 1)
+        )
+        (path "/253d96fc-e3e7-475c-97d3-54a32a6a1970/562c3ef4-3faf-4a2b-b183-c065b2c5f1b8"
+          (reference "J7") (unit 1)
+        )
+      )

Commit message: Add files via upload
Other:
- note added: "connectors for footswitchs"
- note added: "for UART"
Changed lines of the file:
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@@
     (stroke (width 0) (type default))
+  )
+  (text "connectors for footswitchs" (at 177.8 167.64 0)
+    (effects (font (size 1.27 1.27)) (justify left bottom))
   )
   (text "ST Connector\n\n\n" (at 186.69 77.47 0)
     (effects (font (size 1.27 1.27)) (justify left bottom))
   )
+  (text " for UART\n" (at 64.77 242.57 0)
+    (effects (font (size 1.27 1.27)) (justify left bottom))
+  )
