File: Electronic Board/footswitch/footswitch.kicad_sch (KiCad schematic)
At the start: 2 parts, among them J9 Conn_01x03, SW2 SW_SPDT

Commit message: Add files via upload
Parts:
- added J2: 4840.2201, CONN_4840.2201_SCH, symbol 2023-12-05_13-09-39:4840.2201
Connections:
- no-connect marks 0 -> 3
Changed lines of the file:
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@@
 (kicad_sch (version 20230121) (generator eeschema)
   (paper "A4")
+  (no_connect (at 118.11 64.77))
+  (no_connect (at 118.11 67.31))
+  (no_connect (at 118.11 62.23))
   (wire (pts (xy 111.76 93.98) (xy 111.76 91.44))
     (stroke (width 0) (type default))
@@
         )
       )
+    )
+  )
+  (symbol (lib_id "2023-12-05_13-09-39:4840.2201") (at 118.11 62.23 0) (unit 1)
+    (in_bom yes) (on_board yes) (dnp no) (fields_autoplaced)
+    (property "Reference" "J2" (at 132.08 64.135 0)
+      (effects (font (size 1.524 1.524)) (justify left))
+    )
+    (property "Value" "4840.2201" (at 132.08 66.675 0)
+      (effects (font (size 1.524 1.524)) (justify left))
+    )
+    (property "Footprint" "CONN_4840.2201_SCH" (at 119.38 53.34 0)
+      (effects (font (size 1.27 1.27) italic) hide)
+    )
+    (property "Datasheet" "4840.2201" (at 118.11 62.23 0)
+      (effects (font (size 1.27 1.27) italic) hide)
+    )
+    (pin "1")
+    (pin "2")
+    (pin "3")
+    (instances
+      (project "footswitch"
+        (path "/ec86ce07-c9cf-435c-96c9-73697d27d8a9"
+          (reference "J2") (unit 1)
+        )
+      )
